File: kicad/esp32c3-smart-board.kicad_sch (KiCad schematic)
At the start: 69 parts, among them J1 USB_C_Receptacle_USB2.0_16P, J3 Conn_01x12_Pin, Q1 FS8205A, Q2 BSS138, Q3 IRLML6401, SW1 SW_Push, SW2 SW_Push, U1 ME6211C33M5G, U2 ESP32-C3, U3 TP4056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

Commit message: Update KiCAD project for revision 1.3
Parts:
- removed R22: 100R, Resistor_SMD:R_0402_1005Metric, symbol Device:R
- AE1: footprint User:ESPRESSIF_ESP32_MIFA_2.4GHz_Right -> RF_Antenna:Texas_SWRA117D_2.4GHz_Right
Connections:
- net U0RX: now also U2.27 (U0RXD/GPIO20)
Other:
- note added: "Addapt R7 and R6 for I2C Fast Mode"
- moved on the sheet: R21
Changed lines of the file:
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@@
 	(title_block
 		(title "ESP32C3 Smart Board")
-		(date "2025-11-09")
-		(rev "2")
+		(date "2025-12-05")
+		(rev "1.3")
 	)
 	(rectangle
@@
 		)
 	)
+	(text "Addapt R7 and R6\nfor I2C Fast Mode"
+		(exclude_from_sim no)
+		(at 233.934 53.848 0)
+		(effects
+			(font
+				(size 1.27 1.27)
+			)
+		)
+	)
 	(text "Decoupling capacitors"
 		(exclude_from_sim no)
@@
 	)
 	(junction
-		(at 185.42 74.93)
-		(diameter 0)
-		(color 0 0 0 0)
-	)
-	(junction
 		(at 273.05 104.14)
 		(diameter 0)
@@
 	)
 	(junction
-		(at 185.42 77.47)
-		(diameter 0)
-		(color 0 0 0 0)
-	)
-	(junction
 		(at 168.91 34.29)
 		(diameter 0)
@@
 	(wire
 		(pts
-			(xy 191.77 53.34) (xy 191.77 55.88)
-		)
-		(stroke
-			(width 0)
-			(type default)
-		)
-	)
-	(wire
-		(pts
 			(xy 105.41 34.29) (xy 105.41 35.56)
 		)
@@
 	(wire
 		(pts
-			(xy 201.93 57.15) (xy 195.58 57.15)
+			(xy 200.66 67.31) (xy 194.31 67.31)
 		)
 		(stroke
@@
 	(wire
 		(pts
-			(xy 191.77 69.85) (xy 185.42 69.85)
+			(xy 185.42 69.85) (xy 200.66 69.85)
 		)
 		(stroke
@@
 	(wire
 		(pts
-			(xy 184.15 74.93) (xy 185.42 74.93)
-		)
-		(stroke
-			(width 0)
-			(type default)
-		)
-	)
-	(wire
-		(pts
 			(xy 48.26 114.3) (xy 41.91 114.3)
 		)
@@
 	(wire
 		(pts
+			(xy 185.42 77.47) (xy 195.58 77.47)
+		)
+		(stroke
+			(width 0)
+			(type default)
+		)
+	)
+	(wire
+		(pts
 			(xy 78.74 153.67) (xy 78.74 154.94)
 		)
@@
 	(wire
 		(pts
-			(xy 191.77 53.34) (xy 201.93 53.34)
-		)
-		(stroke
-			(width 0)
-			(type default)
-		)
-	)
-	(wire
-		(pts
 			(xy 219.71 25.4) (xy 222.25 25.4)
 		)
@@
 	(wire
 		(pts
-			(xy 195.58 67.31) (xy 185.42 67.31)
+			(xy 186.69 67.31) (xy 185.42 67.31)
 		)
 		(stroke
@@
 	(wire
 		(pts
-			(xy 195.58 66.04) (xy 195.58 67.31)
+			(xy 25.4 85.09) (xy 25.4 77.47)
 		)
 		(stroke
@@
 	(wire
 		(pts
-			(xy 25.4 85.09) (xy 25.4 77.47)
+			(xy 146.05 144.78) (xy 146.05 149.86)
 		)
 		(stroke
@@
 	(wire
 		(pts
-			(xy 146.05 144.78) (xy 146.05 149.86)
+			(xy 185.42 74.93) (xy 195.58 74.93)
 		)
 		(stroke
@@
 	(wire
 		(pts
-			(xy 191.77 63.5) (xy 191.77 69.85)
-		)
-		(stroke
-			(width 0)
-			(type default)
-		)
-	)
-	(wire
-		(pts
 			(xy 252.73 133.35) (xy 255.27 133.35)
 		)
@@
 	(wire
 		(pts
-			(xy 185.42 77.47) (xy 195.58 77.47)
-		)
-		(stroke
-			(width 0)
-			(type default)
-		)
-	)
-	(wire
-		(pts
 			(xy 168.91 24.13) (xy 179.07 24.13)
 		)
@@
 	(wire
 		(pts
-			(xy 184.15 77.47) (xy 185.42 77.47)
-		)
-		(stroke
-			(width 0)
-			(type default)
-		)
-	)
-	(wire
-		(pts
 			(xy 165.1 163.83) (xy 165.1 173.99)
 		)
@@
 	(wire
 		(pts
-			(xy 195.58 57.15) (xy 195.58 58.42)
-		)
-		(stroke
-			(width 0)
-			(type default)
-		)
-	)
-	(wire
-		(pts
 			(xy 41.91 121.92) (xy 49.53 121.92)
 		)
@@
 	(wire
 		(pts
-			(xy 185.42 74.93) (xy 195.58 74.93)
-		)
-		(stroke
-			(width 0)
-			(type default)
-		)
-	)
-	(wire
-		(pts
 			(xy 34.29 74.93) (xy 16.51 74.93)
 		)
@@
 	)
 	(label "U0RX"
-		(at 201.93 53.34 180)
+		(at 200.66 69.85 180)
 		(effects
 			(font
@@
 	)
 	(label "U0TX"
-		(at 201.93 57.15 180)
+		(at 200.66 67.31 180)
 		(effects
 			(font
@@
 			)
 		)
-		(property "Footprint" "User:ESPRESSIF_ESP32_MIFA_2.4GHz_Right"
+		(property "Footprint" "RF_Antenna:Texas_SWRA117D_2.4GHz_Right"
 			(at 53.34 19.05 0)
 			(effects
@@
 	(symbol
 		(lib_id "Device:R")
-		(at 195.58 62.23 180)
+		(at 190.5 67.31 90)
 		(unit 1)
 		(exclude_from_sim no)
@@
 		(fields_autoplaced yes)
 		(property "Reference" "R21"
-			(at 198.12 60.9599 0)
+			(at 190.5 60.96 90)
 			(effects
 				(font
 					(size 1.27 1.27)
 				)
-				(justify right)
 			)
 		)
 		(property "Value" "100R"
-			(at 198.12 63.4999 0)
+			(at 190.5 63.5 90)
 			(effects
 				(font
 					(size 1.27 1.27)
 				)
-				(justify right)
 			)
 		)
 		(property "Footprint" "Resistor_SMD:R_0402_1005Metric"
-			(at 197.358 62.23 90)
+			(at 190.5 69.088 90)
 			(effects
 				(font
@@
 		)
 		(property "Datasheet" "~"
-			(at 195.58 62.23 0)
+			(at 190.5 67.31 0)
 			(effects
 				(font
@@
 		)
 		(property "Description" "Resistor"
-			(at 195.58 62.23 0)
+			(at 190.5 67.31 0)
 			(effects
 				(font
@@
 					(unit 1)
 				)
-			)
-		)
-	)
-	(symbol
-		(lib_id "Device:R")
-		(at 191.77 59.69 0)
-		(mirror x)
-		(unit 1)
-		(exclude_from_sim no)
-		(in_bom yes)
-		(on_board yes)
-		(dnp no)
-		(property "Reference" "R22"
-			(at 189.23 60.9601 0)
-			(effects
-				(font
-					(size 1.27 1.27)
-				)
-				(justify right)
-			)
-		)
-		(property "Value" "100R"
-			(at 189.23 58.4201 0)
-			(effects
-				(font
-					(size 1.27 1.27)
-				)
-				(justify right)
-			)
-		)
-		(property "Footprint" "Resistor_SMD:R_0402_1005Metric"
-			(at 189.992 59.69 90)
-			(effects
-				(font
-					(size 1.27 1.27)
-				)
-				(hide yes)
-			)
-		)
-		(property "Datasheet" "~"
-			(at 191.77 59.69 0)
-			(effects
-				(font
-					(size 1.27 1.27)
-				)
-				(hide yes)
-			)
-		)
-		(property "Description" "Resistor"
-			(at 191.77 59.69 0)
-			(effects
-				(font
-					(size 1.27 1.27)
-				)
-				(hide yes)
-			)
-		)
-		(pin "2"
-		)
-		(pin "1"
-		)
-		(instances
-			(project ""
-				(path "/d9fab985-9caf-4e8c-a371-ec94c3762aca"
-					(reference "R22")
-					(unit 1)
-				)
